Commit message: delete car collision tag

File: urdf/turtlebot3_description/turtlebot3_burger.urdf.xacro (robot description, xacro)
@@ -18,10 +18,4 @@
       <material name="dark"/>
     </visual>
-    <collision>
-      <origin xyz="-0.032 0 0.070" rpy="0 0 0"/>
-      <geometry>
-        <box size="0.140 0.140 0.140"/>
-      </geometry>
-    </collision>
     <inertial>
       <origin xyz="-0.032 0 0" rpy="0 0 0"/>
@@ -45,11 +39,4 @@
       <material name="white"/>
     </visual>
-    <collision>
-      <origin xyz="-0.032 0 0.07" rpy="0 0 0"/>
-      <max_contacts>100</max_contacts>
-      <geometry>
-        <cylinder length="0.02" radius="0.12"/>
-      </geometry>
-    </collision>
     <inertial>
       <origin xyz="-0.032 0 0" rpy="0 0 0"/>
@@ -155,10 +142,4 @@
       <material name="dark"/>
     </visual>
-    <collision>
-      <origin xyz="0 0 0" rpy="0 0 0"/>
-      <geometry>
-        <cylinder length="0.04" radius="0.05"/>
-      </geometry>
-    </collision>
     <inertial>
       <mass value="0.01" />
